File: picochet-scorpion2.kicad_pcb (KiCad board)
At the start: 4 copper layers, 97.2 x 55.6 mm, 55 parts, among them J1 Conn_02x02, J2 Conn_01x02, J3 Conn_01x04, J4 Conn_01x02, J6 Conn_01x05, J8 Conn_01x05, Q1 DMT12H060LFDF, SW1 SW_Push, SW2 SW_Push, SW3 SW_SP3T_Shielded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

Commit message: v0.1 prototype
Parts:
- added QR*****: https://github.com/eatnooM/picochet-scorpion2, rp2354_openfire:picochet-scorpion2-repo-qr, B.Cu at (162.3, 101.6)
- added REF**: OSHW-Logo_7.5x8mm_SilkScreen, Symbol:OSHW-Logo_7.5x8mm_SilkScreen, B.Cu at (153.6, 80.3)
- moved REF** 2.90 mm to (115.1, 79.7)
- moved J3 0.50 mm to (175.4, 118.3)
- moved C21 0.35 mm to (177.7, 107.5)
- moved F1 0.35 mm to (177.7, 111.4)
- moved C1 0.15 mm to (175.4, 104.2)
- moved D1 0.15 mm to (175.4, 108.4)
- moved Q1 0.10 mm to (163.8, 106.8)
- moved R14 0.09 mm to (164.1, 101.8)
- moved R15 0.09 mm to (164.1, 103.5)
Routing:
- net VBUS: track 5.06 -> 5.97 mm
- net /USB_D+: track 61.8 -> 62.3 mm
Other:
- board size 97.2 x 55.6 mm -> 96.7 x 55.6 mm
- board text added: "Mtr"
- board text added: "Picochet-Scorpion2 v0.1 prototype"
- board text added: "Sw."
