File: picochet-scorpion2.kicad_pcb (KiCad board)
At the start: 4 copper layers, 96.7 x 55.6 mm, 57 parts, among them J1 Conn_02x02, J2 Conn_01x02, J3 Conn_01x04, J4 Conn_01x02, J6 Conn_01x05, J8 Conn_01x05, Q1 DMT12H060LFDF, SW1 SW_Push, SW2 SW_Push, SW3 SW_SP3T_Shielded, SW4 SW_Push, SW5 SW_Push, SW6 SW_Push, SW7 SW_SPDT_Shielded, SW8 SW_SPDT_Shielded, U1 RP2354A, U2 NCP1117-3.3_SOT223, Y1 ABM8-272-T3

Commit message: v0.3 WIP
Parts:
- removed JP1: Jumper_2_Open, Jumper:SolderJumper-3_P1.3mm_Open_RoundedPad1.0x1.5mm_NumberLabels
- D1: footprint Diode_SMD:D_SOD-323F -> Diode_SMD:D_SOD-323
- J4: value Conn_01x02 -> Conn_01x03; footprint Connector_PinHeader_2.54mm:PinHeader_1x02_P2.54mm_Vertical -> Connector_PinHeader_2.54mm:PinHeader_1x03_P2.54mm_Vertical
- Q1: value DMT12H060LFDF -> AO3400A; footprint Package_DFN_QFN:Diodes_UDFN2020-6_Type-F -> Package_TO_SOT_SMD:SOT-23
- R14: value 1K -> 100R
- R15: value 100K -> 10K
- SW7, SW8: value SW_SPDT_Shielded -> SW_DPDT; footprint scorpion2:ModeSwitch-SPDT-MountingPoints -> scorpion2:Switch-DPDT-5.8x5.8mm
- moved J4 2.65 mm to (152.0, 120.0)
- moved C1 2.10 mm to (175.4, 102.1)
- moved D1 1.90 mm to (173.5, 108.4)
- moved C21 1.80 mm to (175.8, 107.5)
- moved F1 1.80 mm to (175.8, 111.4)
- moved J3 1.58 mm to (173.9, 118.8)
- moved SW3 1.00 mm to (163.1, 81.9)
- moved R14 0.73 mm to (163.4, 101.6)
- moved R15 0.73 mm to (163.4, 103.3)
- moved Q1 0.50 mm to (163.8, 106.3), turned to -90 degrees
- moved SW7 0.20 mm to (126.1, 89.0), turned to 90 degrees
- turned SW8 to 90 degrees
Connections:
- D3 pad 2: /LED_GND -> GND
- Q1 pad 1: /RMB_GND -> Net-(Q1-G)
- Q1 pad 2: /RMB_GND -> GND
- Q1 pad 3: Net-(Q1-G) -> /RMB_GND
- SW7 pad 1: GND -> (no net)
- SW7 pad 2: /~{FRONT_SW} -> (no net)
- SW7 pad 3: unconnected-(SW7-Pad3) -> (no net)
- SW8 pad 1: GND -> (no net)
- SW8 pad 2: /~{BACK_SW} -> (no net)
- SW8 pad 3: unconnected-(SW8-Pad3) -> (no net)
- U1 pad 15: /~{FRONT_SW} -> /~{BTN_START}
- U1 pad 2: /~{BACK_SW} -> /~{BTN_SELECT}
- U1 pad 8: /LED_DI -> /~{BTN_PEDAL_ALT}
- U1 pad 9: unconnected-(U1-GPIO6-Pad9) -> /LED_DI
Routing:
- net /~{BTN_PEDAL_ALT}: track 0.00 -> 49.2 mm
- net /~{FRONT_SW}: track 38.2 -> 0.00 mm, vias 2 -> 0
- net /~{BTN_SELECT}: track 0.00 -> 10.4 mm
- net /~{BACK_SW}: track 9.14 -> 0.00 mm
- net /~{BTN_START}: track 0.00 -> 8.28 mm, vias 0 -> 1
- net /LED_GND: track 5.46 -> 0.00 mm, vias 1 -> 0
- net /LED_DI: track 45.2 -> 43.0 mm
- net /~{BTN_PEDAL}: track 49.4 -> 47.4 mm
- net VSYS: track 90.4 -> 91.8 mm
- net /~{BTN_TRIGGER}: track 49.9 -> 50.6 mm
- net /RUMBLE: track 37.1 -> 37.8 mm
- net /USB_D-: track 62.4 -> 61.8 mm
- net /USB_D+: track 62.3 -> 61.7 mm
- net /~{BTN_HOME}: track 61.0 -> 61.6 mm
- net GND: vias 71 -> 75
Other:
- board size 96.7 x 55.6 mm -> 94.7 x 55.6 mm
- board text added: "1"
- board text added: "2"
- board text added: "Picochet-Scorpion2 v0.2 prototype"
- board text added: "Select"
- board text added: "Start"
- board text removed: "Always"
- board text removed: "If SW7 on"
- board text removed: "Neopixel power"
- board text removed: "Picochet-Scorpion2 v0.1 prototype"

Commit message: Cost optomise for pcba (#1)
* Cost optomise BOM and PCB layout for PCBA

* Cost optomise

* Change R7 & R8 to 33Ohm 0402 parts (correct issue of 27K)
Parts:
- removed QR*****: https://github.com/eatnooM/picochet-scorpion2, rp2354_openfire:picochet-scorpion2-repo-qr
- removed the REF** at (153.6, 80.3)
- added C25: 100nF, Capacitor_SMD:C_0402_1005Metric, F.Cu at (172.4, 96.9)
- C1, C21: footprint Capacitor_SMD:C_0805_2012Metric_Pad1.18x1.45mm_HandSolder -> Capacitor_SMD:C_0603_1608Metric
- C10, C11, C12, C14, C15, C17, C20, C23, C8, C9: footprint Capacitor_SMD:C_0402_1005Metric_Pad0.74x0.62mm_HandSolder -> Capacitor_SMD:C_0402_1005Metric
- C13, C16, C18, C6, C7: footprint Capacitor_SMD:C_0402_1005Metric_Pad0.74x0.62mm_HandSolder -> Capacitor_SMD:C_0402_1005Metric; moved to F.Cu
- C19, C24, C5: footprint Capacitor_SMD:C_0805_2012Metric_Pad1.18x1.45mm_HandSolder -> Capacitor_SMD:C_0402_1005Metric
- C3, C4: value 15pF -> 30pF; footprint Capacitor_SMD:C_0402_1005Metric_Pad0.74x0.62mm_HandSolder -> Capacitor_SMD:C_0402_1005Metric
- D1: value D_Schottky -> 1N5819WS
- D2: value RBR3LAM60B -> BAT43WS; footprint Diode_SMD:D_SOD-128 -> Diode_SMD:D_SOD-323
- L1, U1: moved to F.Cu
- R14: value 100R -> 100; footprint Resistor_SMD:R_0402_1005Metric_Pad0.72x0.64mm_HandSolder -> Resistor_SMD:R_0402_1005Metric
- R15: value 10K -> 10k; footprint Resistor_SMD:R_0402_1005Metric_Pad0.72x0.64mm_HandSolder -> Resistor_SMD:R_0402_1005Metric
- R2, R6: value 1K -> 1k; footprint Resistor_SMD:R_0402_1005Metric_Pad0.72x0.64mm_HandSolder -> Resistor_SMD:R_0402_1005Metric
- R4: value 1K -> 1k; footprint Resistor_SMD:R_0402_1005Metric_Pad0.72x0.64mm_HandSolder -> Resistor_SMD:R_0402_1005Metric; moved to F.Cu
- R5: value 33R -> 33; footprint Resistor_SMD:R_0402_1005Metric_Pad0.72x0.64mm_HandSolder -> Resistor_SMD:R_0402_1005Metric; moved to F.Cu
- R7, R8: value 27R -> 33; footprint Resistor_SMD:R_0402_1005Metric_Pad0.72x0.64mm_HandSolder -> Resistor_SMD:R_0402_1005Metric; moved to F.Cu
- SW1, SW2: footprint scorpion2:Switch-Push-SMD-4mmx3mm -> Button_Switch_SMD:SW_Push_1P1T_XKB_TS-1187A; moved to F.Cu
- U2: value NCP1117-3.3_SOT223 -> AMS1117-3.3
- Y1: value ABM8-272-T3 -> X322512MSB4SI; footprint Crystal:Crystal_SMD_3225-4Pin_3.2x2.5mm_HandSoldering -> Crystal:Crystal_SMD_3225-4Pin_3.2x2.5mm; moved to F.Cu
- moved SW2 41.3 mm to (146.3, 75.2)
- moved R4 40.9 mm to (141.9, 74.4)
- moved C19 27.8 mm to (143.2, 84.4), turned to -90 degrees
- moved C3 22.0 mm to (147.3, 83.3), turned to -125 degrees
- moved C4 20.1 mm to (147.7, 78.9), turned to 145 degrees
- moved R6 19.9 mm to (125.8, 78.5), turned to 0 degrees
- moved SW1 19.8 mm to (126.8, 81.8)
- moved Y1 18.2 mm to (145.4, 81.4), turned to 55 degrees
- moved L1 16.3 mm to (128.2, 77.1)
- moved R2 13.9 mm to (143.9, 79.2), turned to 55 degrees
- moved C18 11.8 mm to (142.2, 83.2)
- moved R7 11.4 mm to (132.3, 80.2), turned to 0 degrees
- moved C7 11.4 mm to (131.0, 77.6), turned to 90 degrees
- moved R8 11.4 mm to (132.3, 79.2), turned to 0 degrees
- moved C16 10.1 mm to (141.9, 76.3), turned to 90 degrees
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Connections:
- C10 pad 1: GND -> +1V1
- C10 pad 2: +1V1 -> GND
- C12 pad 1: GND -> +3V3
- C12 pad 2: +3V3 -> GND
- C13 pad 1: GND -> +3V3
- C13 pad 2: +3V3 -> GND
- C14 pad 1: GND -> +3V3
- C14 pad 2: +3V3 -> GND
- C15 pad 1: GND -> +3V3
- C15 pad 2: +3V3 -> GND
- C16 pad 1: GND -> +3V3
- C16 pad 2: +3V3 -> GND
- C18 pad 1: GND -> +3V3
- C18 pad 2: +3V3 -> GND
- C20 pad 1: GND -> +3V3
- C20 pad 2: +3V3 -> GND
- C23 pad 1: GND -> VSYS
- C23 pad 2: VSYS -> GND
- C24 pad 1: /RMB_GND -> +3V3
- C24 pad 2: +3V3 -> /RMB_GND
- C6 pad 1: GND -> +3V3
- C6 pad 2: +3V3 -> GND
- C7 pad 1: GND -> +1V1
- C7 pad 2: +1V1 -> GND
- C9 pad 1: GND -> VREG_AVDD
- C9 pad 2: VREG_AVDD -> GND
- R15 pad 1: GND -> Net-(Q1-G)
- R15 pad 2: Net-(Q1-G) -> GND
- R2 pad 1: Net-(C4-Pad2) -> Net-(U1-XOUT)
- R2 pad 2: Net-(U1-XOUT) -> Net-(C4-Pad2)
Routing:
- net +3V3: track 19.1 -> 159.7 mm, vias 39 -> 37
- net /~{RESET}: track 32.3 -> 9.86 mm, vias 2 -> 0
- net /USB_D-: track 61.8 -> 81.0 mm, vias 1 -> 2
- net /USB_D+: track 61.7 -> 80.7 mm, vias 1 -> 2
- net +1V1: track 12.6 -> 25.0 mm, vias 8 -> 4
- net /~{BTN_HOME}: track 61.6 -> 50.7 mm, vias 4 -> 1
- net /~{BTN_A}: track 20.9 -> 30.7 mm, vias 1 -> 2
- net /~{BTN_B}: track 21.5 -> 30.8 mm, vias 2 -> 1
- net /CAM_CLK: track 40.8 -> 49.7 mm, vias 1 -> 2
- net /~{BTN_START}: track 8.28 -> 17.1 mm, vias 1 -> 2
- net /CAM_SDA: track 40.8 -> 48.9 mm, vias 1 -> 2
- net /CAM_SCL: track 42.2 -> 49.5 mm, vias 1 -> 2
- net Net-(U1-~{QSPI_SS}): track 17.3 -> 10.0 mm
- net /VREG_LX: track 0.00 -> 6.42 mm, vias 0 -> 2
- net GND: track 1.42 -> 6.94 mm, vias 75 -> 57
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- added copper zone on B.Cu, net +3V3
- removed copper zone on B.Cu, net (none)
- removed copper zone on B.Cu, net +1V1
- removed copper zone on In2.Cu, net +1V1
- removed copper zone on In1.Cu, net +3V3
- removed copper zone on B.Cu, net /VREG_LX
- removed copper zone on In1.Cu, net GND
- removed copper zone on In2.Cu, net GND
Other:
- copper layers 4 -> 2
- board text removed: "Boot"
