File: picochet-scorpion2.kicad_sch (KiCad schematic)
At the start: 64 parts, among them J1 Conn_02x02, J2 Conn_01x02, J3 Conn_01x04, J4 Conn_01x03, J6 Conn_01x05, J8 Conn_01x05, Q1 AO3400A, SW1 SW_Push, SW2 SW_Push, SW3 SW_SP3T_Shielded, SW4 SW_Push, SW5 SW_Push, SW6 SW_Push, SW7 SW_DPDT, SW8 SW_DPDT, U1 RP2354A, U2 NCP1117-3.3_SOT223, U3 DNF, U4 DNF, Y1 ABM8-272-T3

Commit message: Cost optomise for pcba (#1)
* Cost optomise BOM and PCB layout for PCBA

* Cost optomise

* Change R7 & R8 to 33Ohm 0402 parts (correct issue of 27K)
Parts:
- removed C1, C19, C21, C5: 10uF, Capacitor_SMD:C_0805_2012Metric_Pad1.18x1.45mm_HandSolder, symbol Device:C
- removed C10, C6, C7, C9: 4.7uF, Capacitor_SMD:C_0402_1005Metric_Pad0.74x0.62mm_HandSolder, symbol Device:C
- removed C11, C12, C13, C14, C15, C16, C17, C18, C20, C23, C8: 100nF, Capacitor_SMD:C_0402_1005Metric_Pad0.74x0.62mm_HandSolder, symbol Device:C
- removed C24: 100nF, Capacitor_SMD:C_0805_2012Metric_Pad1.18x1.45mm_HandSolder, symbol Device:C
- removed C3, C4: 15pF, Capacitor_SMD:C_0402_1005Metric_Pad0.74x0.62mm_HandSolder, symbol Device:C
- removed D1: D_Schottky, Diode_SMD:D_SOD-323, symbol Device:D_Schottky
- removed D2: RBR3LAM60B, Diode_SMD:D_SOD-128, symbol Device:D
- removed Q1: AO3400A, Package_TO_SOT_SMD:SOT-23, symbol Transistor_FET:AO3400A
- removed R14: 100R, Resistor_SMD:R_0402_1005Metric_Pad0.72x0.64mm_HandSolder, symbol Device:R
- removed R15: 10K, Resistor_SMD:R_0402_1005Metric_Pad0.72x0.64mm_HandSolder, symbol Device:R
- removed R2, R4, R6: 1K, Resistor_SMD:R_0402_1005Metric_Pad0.72x0.64mm_HandSolder, symbol Device:R
- removed R5: 33R, Resistor_SMD:R_0402_1005Metric_Pad0.72x0.64mm_HandSolder, symbol Device:R
- removed R7, R8: 27R, Resistor_SMD:R_0402_1005Metric_Pad0.72x0.64mm_HandSolder, symbol Device:R
- removed U2: NCP1117-3.3_SOT223, Package_TO_SOT_SMD:SOT-223-3_TabPin2, symbol Regulator_Linear:NCP1117-3.3_SOT223
- added C1, C21: 10uF, Capacitor_SMD:C_0603_1608Metric, symbol JLCPCB_Basic_Capacitor_MLCC:10uF_0603_25V_X5R_±20%
- added C10, C6, C7, C9: 4.7uF, Capacitor_SMD:C_0402_1005Metric, symbol JLCPCB_Basic_Capacitor_MLCC:4.7uF_0402_10V_X5R_±20%
- added C11, C12, C13, C14, C15, C16, C17, C18, C20, C23, C24, C25, C8: 100nF, Capacitor_SMD:C_0402_1005Metric, symbol JLCPCB_Basic_Capacitor_MLCC:100nF_0402_50V_X7R_±10%
- added C19, C5: 10uF, Capacitor_SMD:C_0402_1005Metric, symbol JLCPCB_Basic_Capacitor_MLCC:10uF_0402_6.3V_X5R_±20%
- added C3, C4: 30pF, Capacitor_SMD:C_0402_1005Metric, symbol JLCPCB_Basic_Capacitor_MLCC:30pF_0402_50V_C0G_±5%
- added D1: 1N5819WS, Diode_SMD:D_SOD-323, symbol JLCPCB_Basic_Diode-Schottky:1N5819WS
- added D2: BAT43WS, Diode_SMD:D_SOD-323, symbol JLCPCB_Basic_Diode-Schottky:BAT43WS
- added Q1: AO3400A, Package_TO_SOT_SMD:SOT-23, symbol JLCPCB_Basic_Mosfet_NPN:AO3400A
- added R14: 100, Resistor_SMD:R_0402_1005Metric, symbol JLCPCB_Basic_Resistor:100Ω_0402_±1%
- added R15: 10k, Resistor_SMD:R_0402_1005Metric, symbol JLCPCB_Basic_Resistor:10kΩ_0402_±1%
- added R2, R4, R6: 1k, Resistor_SMD:R_0402_1005Metric, symbol JLCPCB_Basic_Resistor:1kΩ_0402_±1%
- added R5, R7, R8: 33, Resistor_SMD:R_0402_1005Metric, symbol JLCPCB_Basic_Resistor:33Ω_0402_±1%
- added U2: AMS1117-3.3, Package_TO_SOT_SMD:SOT-223-3_TabPin2, symbol Regulator_Linear:AMS1117-3.3
- D3: LCSC (none) -> C42417498
- F1: LCSC (none) -> C269104
- L1: LCSC (none) -> C42411119
- SW1, SW2: footprint scorpion2:Switch-Push-SMD-4mmx3mm -> Button_Switch_SMD:SW_Push_1P1T_XKB_TS-1187A; LCSC (none) -> C318884; LCSC Part # C455280 -> (none)
- SW7, SW8: LCSC (none) -> C22459505
- U1: LCSC (none) -> C41378174
- Y1: value ABM8-272-T3 -> X322512MSB4SI; footprint Crystal:Crystal_SMD_3225-4Pin_3.2x2.5mm_HandSoldering -> Crystal:Crystal_SMD_3225-4Pin_3.2x2.5mm; LCSC (none) -> C9002; LCSC Part # C20625731 -> (none)
Connections:
- net +1V1: now also C10.1, C11.2, C7.1, C8.2
- net +3V3: now also C12.1, C13.1, C14.1, C15.1, C16.1, C17.1, C18.1, C19.1, C20.1, C24.1, C25.2, C5.1, C6.1, D2.1 (K), R5.1, U2.2 (VO)
- net +5V: now also C21.1, D1.2 (A)
- net GND: now also C1.2, C10.2, C11.1, C12.2, C13.2, C14.2, C15.2, C16.2, C17.2, C18.2, C19.2, C20.2, C21.2, C23.2, C25.1, C3.1, C4.1, C5.2, C6.2, C7.2, C8.1, C9.2, Q1.2 (S), R15.2, R4.1, R6.1, U2.1 (GND)
- net RMB_GND: now also C24.2, D2.2 (A), Q1.3 (D)
- net RUMBLE: now also R14.1
- net USB_D+: now also R7.1
- net USB_D-: now also R8.1
- net VREG_AVDD: now also C9.1, R5.2
- net VSYS: now also C1.1, C23.1, D1.1 (K), U2.3 (VI)
- net at U1.52 (USB_DP): now also R7.2
- net at Y1.3: now also C4.2, R2.2
- net at SW2.1: now also R4.2
- net at SW1.1: now also R6.2
- net at U1.21 (XIN), Y1.1: now also C3.2
- net at U1.22 (XOUT): now also R2.1
- net at U1.51 (USB_DM): now also R8.2
- new net: Q1.1 (G), R14.2, R15.1
Other:
- moved on the sheet: L1
